File: led_array_mixed/led_array.kicad_pcb (KiCad board)
At the start: 2 copper layers, 32 x 32 mm, 66 parts, among them P1 CONN_8, P2 CONN_8

Commit message: Added note about inverting labels.
Other:
- board text added: "Need to invert label - TOP is bottom and BOTTOM is top. Also, invert writting."
Changed lines of the file:
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@@
-(kicad_pcb (version 3) (host pcbnew "(2013-mar-13)-testing")
+(kicad_pcb (version 3) (host pcbnew "(2013-jul-07)-stable")
   (general
     (links 128)
@@
     (area 50.374674 49.8729 85.280114 82.989421)
     (thickness 1.6002)
-    (drawings 7)
+    (drawings 8)
     (tracks 724)
     (zones 0)
@@
   )
   (page A4)
-  (title_block
-    (date "12 feb 2013")
-  )
   (layers
     (15 Front signal)
@@
     )
   )
+  (gr_text "Need to invert label - TOP is bottom and BOTTOM is top. Also, invert writting." (at 75 90) (layer Dwgs.User)
+    (effects (font (size 2.032 1.524) (thickness 0.3048)))
+  )
   (gr_text "Mixed UV/Green \n8x8 LED Array V0.1\nwww.iorodeo.com" (at 65.1 66.8 90) (layer B.SilkS)
     (effects (font (size 1.016 1.016) (thickness 0.2032)) (justify mirror))
@@
   )
   (gr_text Top (at 52.45 66.35 90) (layer B.SilkS)
-    (effects (font (thickness 0.2032)) (justify mirror))
+    (effects (font (size 1.524 1.524) (thickness 0.2032)) (justify mirror))
   )
   (gr_line (start 50.8 50.8) (end 50.8 82.79892) (angle 90) (layer Edge.Cuts) (width 0.381))

Commit message: Added gerber files for version 0.2 of the design.  In version 0.1 the TOP and BOTTOM labels where swapped. Version 0.2 corrects this issue.
Other:
- board text added: "Mixed UV/Green 8x8 LED Array V0.2 www.iorodeo.com"
- board text removed: "Mixed UV/Green 8x8 LED Array V0.1 www.iorodeo.com"
- board text removed: "Need to invert label - TOP is bottom and BOTTOM is top. Also, invert writting."
Changed lines of the file:
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@@
     (links 128)
     (no_connects 0)
-    (area 50.374674 49.8729 85.280114 82.989421)
+    (area 48.819886 49.8729 83.224226 82.989421)
     (thickness 1.6002)
-    (drawings 8)
+    (drawings 7)
     (tracks 724)
     (zones 0)
@@
       (drillshape 0)
       (scaleselection 1)
-      (outputdirectory gerber_v0p1/))
+      (outputdirectory gerber_v0p2/))
   )
   (net 0 "")
@@
     )
   )
-  (gr_text "Need to invert label - TOP is bottom and BOTTOM is top. Also, invert writting." (at 75 90) (layer Dwgs.User)
-    (effects (font (size 2.032 1.524) (thickness 0.3048)))
-  )
-  (gr_text "Mixed UV/Green \n8x8 LED Array V0.1\nwww.iorodeo.com" (at 65.1 66.8 90) (layer B.SilkS)
+  (gr_text "Mixed UV/Green \n8x8 LED Array V0.2\nwww.iorodeo.com" (at 69 66 270) (layer B.SilkS)
     (effects (font (size 1.016 1.016) (thickness 0.2032)) (justify mirror))
   )
-  (gr_text Bottom (at 81.1 67.1 90) (layer B.SilkS)
+  (gr_text Bottom (at 53 67 270) (layer B.SilkS)
     (effects (font (size 2.032 1.524) (thickness 0.3048)) (justify mirror))
   )
-  (gr_text Top (at 52.45 66.35 90) (layer B.SilkS)
+  (gr_text Top (at 81 68 270) (layer B.SilkS)
     (effects (font (size 1.524 1.524) (thickness 0.2032)) (justify mirror))
   )
